File: Mumo.kicad_pcb (KiCad board)
At the start: 4 copper layers, 18 x 13 mm, 25 parts, among them J1 TOP_PINS, J2 BOTTOM_PINS, U1 QMC6309, U2 ICM45686, U3 1532H

Commit message: v1.2 -  use QMC6309H, bridge 5-8 by default
Parts:
- U1: value QMC6309 -> QMC6309H
- renumbered JP5 to JP1, JP6 to JP2, JP7 to JP3, JP8 to JP4, JP4 to JP5, JP2 to JP6, JP1 to JP7, JP3 to JP8
