File: Mumo.kicad_sch (KiCad schematic)
At the start: 19 parts, among them J1 Top_Pins, J2 Bottom Pins, U1 QMC6309, U2 ICM45686, U3 1532H

Commit message: v1.1
Parts:
- added JP1: SDX_AUX_JMP, Mumo Footprints:JMP_CLSD, symbol Mumo Symbols:SolderJumper_2_Bridged
- added JP2: SCX_PU_JMP, Mumo Footprints:JMP_CLSD, symbol Mumo Symbols:SolderJumper_2_Bridged
- added JP3: SDX_PU_JMP, Mumo Footprints:JMP_CLSD, symbol Mumo Symbols:SolderJumper_2_Bridged
- added JP4: SCX_AUX_JMP, Mumo Footprints:JMP_CLSD, symbol Mumo Symbols:SolderJumper_2_Bridged
- J1: value Top_Pins -> TOP_PINS
- J2: value Bottom Pins -> BOTTOM_PINS; symbol Connector:Conn_01x06_Socket -> Mumo Symbols:Conn_01x06_Socket
- JP5: renamed from JP1; value JMP -> SCL_PU_JMP; symbol Jumper:SolderJumper_2_Bridged -> Mumo Symbols:SolderJumper_2_Bridged
- JP6: renamed from JP2; value JMP -> SDA_PU_JMP; symbol Jumper:SolderJumper_2_Bridged -> Mumo Symbols:SolderJumper_2_Bridged
- JP7: renamed from JP3; value JMP -> CS_PU_JMP; symbol Jumper:SolderJumper_2_Bridged -> Mumo Symbols:SolderJumper_2_Bridged
- JP8: renamed from JP4; value JMP -> SD0_PU_JMP; symbol Jumper:SolderJumper_2_Bridged -> Mumo Symbols:SolderJumper_2_Bridged
- JP9: renamed from JP5; value SD0_JMP -> SD0_GND_JMP; symbol Jumper:SolderJumper_2_Open -> Mumo Symbols:SolderJumper_2_Open
Connections:
- net SCX: now also JP2.1 (A), JP4.2 (B); no longer R1.2, U2.3 (ASCx)
- net SDX: now also JP1.2 (B), JP3.1 (A); no longer R2.2, U2.2 (ASDx)
- new net: JP3.2 (B), R2.2
- new net: JP2.2 (B), R1.2
- new net: JP4.1 (A), U2.3 (ASCx)
- new net: JP1.1 (A), U2.2 (ASDx)
Other:
- note added: "Jumper 1: Connects 4k7R pull-up to +3v3 for the SCL pin"
- note added: "Jumper 2: Connects 4k7R pull-up to +3v3 for the SDA pin"
- note added: "Jumper 3: Connects 4k7R pull-up to +3v3 for the CS pin"
- note added: "Jumper 4: Connects 4k7R pull-up to +3v3 for the SD0 pin"
- note added: "Jumper 5: Connects the magnetometer's SCL pin to the IMU's SCX pin"
- note added: "Jumper 6: Connects 10kR pull-up to +3v3 for SCX"
- note added: "Jumper 7: Connects the magnetometer's SDA pin to the IMU's SDX pin"
- note added: "Jumper 8: Connects 10kR pull-up to +3v3 for SDX"
- note added: "Jumper 9: Connects SD0 to GND"
- moved on the sheet: C3, R1, R2, R4, R5, R6, U1
